Commit message: add of  pilote and controle code

File: models/agri_hexacopter.urdf (robot description, URDF)
Before this commit: robot agri_hexacopter_pro_v2, 32 links, 31 joints
Links:
- removed link arm_1
- removed link arm_2
- removed link arm_3
- removed link arm_4
- removed link arm_5
- removed link arm_6
- removed link flowmeter
- removed link foot_left
- removed link foot_right
- removed link leg_left
- removed link leg_right
- removed link lidar_sensor
- removed link motor_1
- removed link motor_2
- removed link motor_3
- removed link motor_4
- removed link motor_5
- removed link motor_6
- removed link nozzle_1
- removed link nozzle_2
- removed link nozzle_3
- removed link nozzle_4
- removed link nozzle_5
- removed link nozzle_6
- removed link rtk_module
- added link agri_payload; visual box size=0.05 0.05 0.03; visual box size=0.22 0.22 0.18
- added link arms_visual; visual box size=1.1 0.04 0.03; visual box size=1.1 0.04 0.03
- added link landing_gear; collision box size=0.6 0.05 0.03; collision box size=0.6 0.05 0.03
- link base_link: mass 6.5 -> 15.0; geometry collision box size=0.3 0.3 0.12; visual cylinder length=0.12 radius=0.25
- link prop_1: geometry visual cylinder length=0.01 radius=0.18
- link prop_2: geometry visual cylinder length=0.01 radius=0.18
- link prop_3: geometry visual cylinder length=0.01 radius=0.18
- link prop_4: geometry visual cylinder length=0.01 radius=0.18
- link prop_5: geometry visual cylinder length=0.01 radius=0.18
- link prop_6: geometry visual cylinder length=0.01 radius=0.18
Joints:
- removed joint joint_arm_1
- removed joint joint_arm_2
- removed joint joint_arm_3
- removed joint joint_arm_4
- removed joint joint_arm_5
- removed joint joint_arm_6
- removed joint joint_flowmeter
- removed joint joint_foot_left
- removed joint joint_foot_right
- removed joint joint_leg_left
- removed joint joint_leg_right
- removed joint joint_lidar
- removed joint joint_motor_1
- removed joint joint_motor_2
- removed joint joint_motor_3
- removed joint joint_motor_4
- removed joint joint_motor_5
- removed joint joint_motor_6
- removed joint joint_nozzle_1
- removed joint joint_nozzle_2
- removed joint joint_nozzle_3
- removed joint joint_nozzle_4
- removed joint joint_nozzle_5
- removed joint joint_nozzle_6
- removed joint joint_prop_1
- removed joint joint_prop_2
- removed joint joint_prop_3
- removed joint joint_prop_4
- removed joint joint_prop_5
- removed joint joint_prop_6
- removed joint joint_rtk
- added joint j_p1: type continuous, parent base_link, child prop_1, origin xyz=0.55 0 0.06, axis 0 0 1
- added joint j_p2: type continuous, parent base_link, child prop_2, origin xyz=-0.55 0 0.06, axis 0 0 1
- added joint j_p3: type continuous, parent base_link, child prop_3, origin xyz=0.27 0.47 0.06, axis 0 0 1
- added joint j_p4: type continuous, parent base_link, child prop_4, origin xyz=-0.27 -0.47 0.06, axis 0 0 1
- added joint j_p5: type continuous, parent base_link, child prop_5, origin xyz=0.27 -0.47 0.06, axis 0 0 1
- added joint j_p6: type continuous, parent base_link, child prop_6, origin xyz=-0.27 0.47 0.06, axis 0 0 1
- added joint joint_arms: type fixed, parent base_link, child arms_visual
- added joint joint_gear: type fixed, parent base_link, child landing_gear
- added joint joint_payload: type fixed, parent base_link, child agri_payload, origin xyz=0 0 0
