Commit message: finalisation

File: models/agri_hexacopter.urdf (robot description, URDF)
Before this commit: robot agri_hexacopter_pro, 10 links, 9 joints
Links:
- link agri_payload: mass None -> 0.0
- link arms_visual: mass None -> 0.0
- link landing_gear: mass None -> 0.0
- link prop_1: mass None -> 0.0
- link prop_2: mass None -> 0.0
- link prop_3: mass None -> 0.0
- link prop_4: mass None -> 0.0
- link prop_5: mass None -> 0.0
- link prop_6: mass None -> 0.0
Joints:
- joint joint_arms: origin (none) -> xyz=0 0 0
- joint joint_gear: origin (none) -> xyz=0 0 0
